File: pcb/keeb_pcb.kicad_pcb (KiCad board)
At the start: 2 copper layers, 355.7 x 122 mm, 242 parts, among them J1 Conn_01x04, SW10 SW_Push, SW11 SW_Push, SW12 SW_Push, SW13 SW_Push, SW14 SW_Push, SW15 SW_Push, SW16 SW_Push, SW17 SW_Push, SW18 SW_Push, SW19 SW_Push, SW2 SW_Push, SW20 SW_Push, SW21 SW_Push, SW22 SW_Push, SW23 SW_Push, SW24 SW_Push, SW25 SW_Push, SW26 SW_Push, SW27 SW_Push, SW29 SW_Push, SW3 SW_Push, SW30 SW_Push, SW31 SW_Push, SW32 SW_Push, SW33 SW_Push, SW34 SW_Push, SW35 SW_Push, SW36 SW_Push, SW37 SW_Push, SW38 SW_Push, SW39 SW_Push, SW4 SW_Push, SW40 SW_Push, SW41 SW_Push, SW42 SW_Push, SW43 SW_Push, SW44 SW_Push, SW45 SW_Push, SW46 SW_Push, SW47 SW_Push, SW48 SW_Push, SW49 SW_Push, SW5 SW_Push, SW50 SW_Push, SW51 SW_Push, SW52 SW_Push, SW53 SW_Push, SW54 SW_Push, SW55 SW_Push, SW57 SW_Push, SW58 SW_Push, SW6 SW_Push, SW60 SW_Push, SW61 SW_Push, SW62 SW_Push, SW63 SW_Push, SW64 SW_Push, SW65 SW_Push, SW66 SW_Push, SW67 SW_Push, SW68 SW_Push, SW69 SW_Push, SW7 SW_Push, SW71 SW_Push, SW72 SW_Push, SW73 SW_Push, SW74 SW_Push, SW77 SW_Push, SW79 SW_Push, SW8 SW_Push, SW80 SW_Push, SW81 SW_Push, SW82 SW_Push, SW9 SW_Push, SW90 SW_Push, SW91 SW_Push, SW92 SW_Push, SW93 SW_Push

Commit message: Added devlog and files for latest journal
Parts:
- SW10, SW11, SW12, SW13, SW14, SW15, SW16, SW17, SW18, SW19, SW2, SW20, SW21, SW22, SW23, SW24, SW25, SW26, SW27, SW29, SW3, SW30, SW31, SW32, SW33, SW34, SW35, SW36, SW37, SW38, SW39, SW4, SW40, SW41, SW42, SW43, SW44, SW45, SW46, SW47, SW48, SW49, SW5, SW50, SW51, SW52, SW53, SW54, SW55, SW57, SW58, SW6, SW60, SW61, SW62, SW63, SW64, SW65, SW66, SW67, SW68, SW69, SW7, SW71, SW72, SW73, SW74, SW77, SW79, SW8, SW80, SW81, SW82, SW9, SW90, SW91, SW92, SW93: footprint PCM_marbastlib-mx:SW_MX_1u -> KeyBoardLibrary:SW_MX_1u
- moved A1 25.7 mm to (305.0, 27.8)
- moved J1 7.62 mm to (345.6, 51.2), turned to -90 degrees
Routing:
- net RGB_D27: track 0.00 -> 342.9 mm
- net +5V: track 130.8 -> 439.3 mm, vias 24 -> 60
- net RGB_D43: track 0.00 -> 288.9 mm, vias 0 -> 4
- net GND: track 2414.4 -> 2449.0 mm
- net /OLED_SDA: track 0.00 -> 18.0 mm
- net /OLED_SCL: track 35.2 -> 25.9 mm, vias 0 -> 2
- net /ROW5: track 443.3 -> 445.4 mm
- net /COL11: track 262.0 -> 264.0 mm
- net /COL13: track 226.8 -> 227.9 mm
Other:
- board size 355.7 x 122 mm -> 359.9 x 124.2 mm
