File: pcb/keeb_pcb.kicad_pcb (KiCad board)
At the start: 2 copper layers, 359.9 x 124.2 mm, 242 parts, among them J1 Conn_01x04, SW10 SW_Push, SW11 SW_Push, SW12 SW_Push, SW13 SW_Push, SW14 SW_Push, SW15 SW_Push, SW16 SW_Push, SW17 SW_Push, SW18 SW_Push, SW19 SW_Push, SW2 SW_Push, SW20 SW_Push, SW21 SW_Push, SW22 SW_Push, SW23 SW_Push, SW24 SW_Push, SW25 SW_Push, SW26 SW_Push, SW27 SW_Push, SW29 SW_Push, SW3 SW_Push, SW30 SW_Push, SW31 SW_Push, SW32 SW_Push, SW33 SW_Push, SW34 SW_Push, SW35 SW_Push, SW36 SW_Push, SW37 SW_Push, SW38 SW_Push, SW39 SW_Push, SW4 SW_Push, SW40 SW_Push, SW41 SW_Push, SW42 SW_Push, SW43 SW_Push, SW44 SW_Push, SW45 SW_Push, SW46 SW_Push, SW47 SW_Push, SW48 SW_Push, SW49 SW_Push, SW5 SW_Push, SW50 SW_Push, SW51 SW_Push, SW52 SW_Push, SW53 SW_Push, SW54 SW_Push, SW55 SW_Push, SW57 SW_Push, SW58 SW_Push, SW6 SW_Push, SW60 SW_Push, SW61 SW_Push, SW62 SW_Push, SW63 SW_Push, SW64 SW_Push, SW65 SW_Push, SW66 SW_Push, SW67 SW_Push, SW68 SW_Push, SW69 SW_Push, SW7 SW_Push, SW71 SW_Push, SW72 SW_Push, SW73 SW_Push, SW74 SW_Push, SW77 SW_Push, SW79 SW_Push, SW8 SW_Push, SW80 SW_Push, SW81 SW_Push, SW82 SW_Push, SW9 SW_Push, SW90 SW_Push, SW91 SW_Push, SW92 SW_Push, SW93 SW_Push

Commit message: Updated with Log 6
Parts:
- added C1: 4.7 uF, Capacitor_SMD:C_0805_2012Metric, F.Cu at (349.0, 64.0)
- added C2: 4.7 uF, Capacitor_SMD:C_0805_2012Metric, F.Cu at (340.0, 65.0)
- added D1: SS14, Diode_SMD:D_SMA, F.Cu at (342.0, 56.0)
- added D94: 1N4148, Diode_THT:D_DO-35_SOD27_P7.62mm_Horizontal, B.Cu at (335.0, 95.0)
- added D95: 1N4148, Diode_THT:D_DO-35_SOD27_P7.62mm_Horizontal, B.Cu at (284.5, 49.0)
- added JST_1: J_BAT, Connector_JST:JST_PH_B2B-PH-K_1x02_P2.00mm_Vertical, F.Cu at (345.0, 82.0)
- added R1: 10k, Resistor_SMD:R_0805_2012Metric, F.Cu at (349.0, 60.0)
- added RGB83: SK6812MINI-E, LED_SMD:LED_SK6812MINI-E_3.2x2.8mm_P1.5mm_ReverseMount, B.Cu at (272.6, 45.1)
- added RGB84: SK6812MINI-E, LED_SMD:LED_SK6812MINI-E_3.2x2.8mm_P1.5mm_ReverseMount, B.Cu at (291.7, 45.1)
- added SW1: SW_PWR, Button_Switch_THT:SW_Slide-03_Wuerth-WS-SLTV_10x2.5x6.4_P2.54mm, F.Cu at (363.0, 65.0)
- added SW94: Programmable 1, KeyBoardLibrary:SW_MX_1u, F.Cu at (272.6, 40.0)
- added SW95: Programmable 2, KeyBoardLibrary:SW_MX_1u, F.Cu at (291.7, 40.0)
- added U1: MCP73831-2-OT, Package_TO_SOT_SMD:SOT-23-5, F.Cu at (345.0, 65.0)
- moved D13 38.1 mm to (234.5, 49.0)
- moved RGB12 38.1 mm to (234.5, 45.1)
- moved SW13 38.1 mm to (234.5, 40.0)
- moved D11 38.1 mm to (196.4, 49.0)
- moved RGB10 38.1 mm to (196.4, 45.1)
- moved SW11 38.1 mm to (196.4, 40.0)
- moved D12 38.1 mm to (215.5, 49.0)
- moved D14 38.1 mm to (246.4, 49.0)
- moved RGB11 38.1 mm to (215.5, 45.1)
- moved RGB13 38.1 mm to (253.6, 45.1)
- moved SW12 38.1 mm to (215.5, 40.0)
- moved SW14 38.1 mm to (253.6, 40.0)
- moved D10 28.6 mm to (177.4, 49.0)
- moved RGB9 28.6 mm to (177.4, 45.1)
- moved SW10 28.6 mm to (177.4, 40.0)
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Connections:
- A1 pad 36: unconnected-(A1-3V3-Pad36)_1 -> +3V3
- A1 pad 39: unconnected-(A1-VSYS-Pad39)_1 -> Net-(A1-VSYS)
- J1 pad 2: +5V -> +3V3
- RGB13 pad 4: RGB_D13 -> RGB_NEW_A
Routing:
- net GND: track 2449.0 -> 2928.5 mm, vias 14 -> 28
- net /COL3: track 629.0 -> 953.7 mm, vias 0 -> 12
- net +5V: track 439.3 -> 693.0 mm, vias 60 -> 73
- net /ROW5: track 445.4 -> 607.4 mm, vias 0 -> 3
- net /COL5: track 315.4 -> 475.2 mm, vias 0 -> 15
- net Net-(D94-A): track 0.00 -> 141.5 mm
- net /COL9: track 252.7 -> 384.9 mm, vias 0 -> 10
- net /COL6: track 303.7 -> 375.3 mm, vias 0 -> 11
- net /ROW0: track 369.3 -> 422.9 mm
- net Net-(D95-A): track 0.00 -> 53.1 mm, vias 0 -> 9
- net /COL2: track 388.9 -> 436.3 mm, vias 0 -> 9
- net /BAT+: track 0.00 -> 45.6 mm, vias 0 -> 1
- net Net-(A1-VSYS): track 0.00 -> 35.1 mm, vias 0 -> 4
- net +3V3: track 0.00 -> 27.2 mm, vias 0 -> 1
- net /BAT_SW: track 0.00 -> 22.7 mm, vias 0 -> 1
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