File: pcb/keeb_pcb.kicad_pcb (KiCad board)
At the start: 2 copper layers, 359.9 x 124.2 mm, 255 parts, among them J1 Conn_01x04, SW1 SW_PWR, SW10 SW_Push, SW11 SW_Push, SW12 SW_Push, SW13 SW_Push, SW14 SW_Push, SW15 SW_Push, SW16 SW_Push, SW17 SW_Push, SW18 SW_Push, SW19 SW_Push, SW2 SW_Push, SW20 SW_Push, SW21 SW_Push, SW22 SW_Push, SW23 SW_Push, SW24 SW_Push, SW25 SW_Push, SW26 SW_Push, SW27 SW_Push, SW29 SW_Push, SW3 SW_Push, SW30 SW_Push, SW31 SW_Push, SW32 SW_Push, SW33 SW_Push, SW34 SW_Push, SW35 SW_Push, SW36 SW_Push, SW37 SW_Push, SW38 SW_Push, SW39 SW_Push, SW4 SW_Push, SW40 SW_Push, SW41 SW_Push, SW42 SW_Push, SW43 SW_Push, SW44 SW_Push, SW45 SW_Push, SW46 SW_Push, SW47 SW_Push, SW48 SW_Push, SW49 SW_Push, SW5 SW_Push, SW50 SW_Push, SW51 SW_Push, SW52 SW_Push, SW53 SW_Push, SW54 SW_Push, SW55 SW_Push, SW57 SW_Push, SW58 SW_Push, SW6 SW_Push, SW60 SW_Push, SW61 SW_Push, SW62 SW_Push, SW63 SW_Push, SW64 SW_Push, SW65 SW_Push, SW66 SW_Push, SW67 SW_Push, SW68 SW_Push, SW69 SW_Push, SW7 SW_Push, SW71 SW_Push, SW72 SW_Push, SW73 SW_Push, SW74 SW_Push, SW77 SW_Push, SW79 SW_Push, SW8 SW_Push, SW80 SW_Push, SW81 SW_Push, SW82 SW_Push, SW9 SW_Push, SW90 SW_Push, SW91 SW_Push, SW92 SW_Push, SW93 SW_Push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

Commit message: Publish checked keyboard hardware, fabrication files and repaired case source
Parts:
- added C10: 1uF, Capacitor_SMD:C_0805_2012Metric, F.Cu at (350.5, 69.5)
- added C101: 100nF, Capacitor_SMD:C_0603_1608Metric, B.Cu at (31.0, 44.1)
- added C102: 100nF, Capacitor_SMD:C_0603_1608Metric, B.Cu at (48.5, 43.1)
- added C103: 100nF, Capacitor_SMD:C_0603_1608Metric, B.Cu at (67.6, 43.1)
- added C104: 100nF, Capacitor_SMD:C_0603_1608Metric, B.Cu at (86.7, 46.1)
- added C105: 100nF, Capacitor_SMD:C_0603_1608Metric, B.Cu at (106.7, 44.1)
- added C106: 100nF, Capacitor_SMD:C_0603_1608Metric, B.Cu at (124.7, 46.1)
- added C107: 100nF, Capacitor_SMD:C_0603_1608Metric, B.Cu at (144.3, 43.6)
- added C108: 100nF, Capacitor_SMD:C_0603_1608Metric, B.Cu at (162.8, 46.1)
- added C109: 100nF, Capacitor_SMD:C_0603_1608Metric, B.Cu at (182.9, 44.1)
- added C110: 100nF, Capacitor_SMD:C_0603_1608Metric, B.Cu at (200.9, 46.1)
- added C111: 100nF, Capacitor_SMD:C_0603_1608Metric, B.Cu at (220.0, 46.1)
- added C112: 100nF, Capacitor_SMD:C_0603_1608Metric, B.Cu at (232.5, 48.6)
- added C113: 100nF, Capacitor_SMD:C_0603_1608Metric, B.Cu at (258.1, 43.1)
- added C114: 100nF, Capacitor_SMD:C_0603_1608Metric, B.Cu at (30.5, 64.7)
- added C115: 100nF, Capacitor_SMD:C_0603_1608Metric, B.Cu at (49.5, 64.7)
- added C116: 100nF, Capacitor_SMD:C_0603_1608Metric, B.Cu at (68.6, 64.7)
- added C117: 100nF, Capacitor_SMD:C_0603_1608Metric, B.Cu at (87.7, 64.7)
- added C118: 100nF, Capacitor_SMD:C_0603_1608Metric, B.Cu at (106.7, 65.7)
- added C119: 100nF, Capacitor_SMD:C_0603_1608Metric, B.Cu at (124.8, 61.7)
- added C120: 100nF, Capacitor_SMD:C_0603_1608Metric, B.Cu at (143.8, 61.7)
- added C121: 100nF, Capacitor_SMD:C_0603_1608Metric, B.Cu at (162.8, 65.2)
- added C122: 100nF, Capacitor_SMD:C_0603_1608Metric, B.Cu at (182.9, 64.7)
- added C123: 100nF, Capacitor_SMD:C_0603_1608Metric, B.Cu at (200.9, 61.7)
- added C124: 100nF, Capacitor_SMD:C_0603_1608Metric, B.Cu at (221.0, 64.7)
- added C125: 100nF, Capacitor_SMD:C_0603_1608Metric, B.Cu at (240.1, 64.7)
- added C126: 100nF, Capacitor_SMD:C_0603_1608Metric, B.Cu at (258.1, 61.7)
- added C127: 100nF, Capacitor_SMD:C_0603_1608Metric, B.Cu at (286.7, 63.7)
- added C128: 100nF, Capacitor_SMD:C_0603_1608Metric, B.Cu at (58.1, 84.2)
- added C129: 100nF, Capacitor_SMD:C_0603_1608Metric, B.Cu at (77.1, 84.2)
- added C130: 100nF, Capacitor_SMD:C_0603_1608Metric, B.Cu at (96.2, 84.2)
- added C131: 100nF, Capacitor_SMD:C_0603_1608Metric, B.Cu at (115.0, 84.2)
- added C132: 100nF, Capacitor_SMD:C_0603_1608Metric, B.Cu at (134.3, 84.2)
- added C133: 100nF, Capacitor_SMD:C_0603_1608Metric, B.Cu at (153.3, 84.2)
- added C134: 100nF, Capacitor_SMD:C_0603_1608Metric, B.Cu at (172.4, 84.2)
- added C135: 100nF, Capacitor_SMD:C_0603_1608Metric, B.Cu at (191.4, 84.2)
- added C136: 100nF, Capacitor_SMD:C_0603_1608Metric, B.Cu at (210.5, 84.2)
- added C137: 100nF, Capacitor_SMD:C_0603_1608Metric, B.Cu at (229.5, 84.2)
- added C138: 100nF, Capacitor_SMD:C_0603_1608Metric, B.Cu at (248.6, 84.2)
- added C139: 100nF, Capacitor_SMD:C_0603_1608Metric, B.Cu at (267.6, 81.8)
- added C140: 100nF, Capacitor_SMD:C_0603_1608Metric, B.Cu at (291.4, 80.8)
- added C141: 100nF, Capacitor_SMD:C_0603_1608Metric, B.Cu at (62.8, 103.3)
- added C142: 100nF, Capacitor_SMD:C_0603_1608Metric, B.Cu at (81.9, 103.3)
- added C143: 100nF, Capacitor_SMD:C_0603_1608Metric, B.Cu at (100.9, 103.3)
- added C144: 100nF, Capacitor_SMD:C_0603_1608Metric, B.Cu at (120.0, 103.3)
- added C145: 100nF, Capacitor_SMD:C_0603_1608Metric, B.Cu at (139.0, 103.3)
- added C146: 100nF, Capacitor_SMD:C_0603_1608Metric, B.Cu at (158.1, 103.3)
- added C147: 100nF, Capacitor_SMD:C_0603_1608Metric, B.Cu at (177.1, 103.3)
- added C148: 100nF, Capacitor_SMD:C_0603_1608Metric, B.Cu at (196.2, 103.3)
- added C149: 100nF, Capacitor_SMD:C_0603_1608Metric, B.Cu at (215.2, 103.3)
- added C150: 100nF, Capacitor_SMD:C_0603_1608Metric, B.Cu at (233.3, 98.8)
- added C151: 100nF, Capacitor_SMD:C_0603_1608Metric, B.Cu at (253.3, 103.3)
- added C152: 100nF, Capacitor_SMD:C_0603_1608Metric, B.Cu at (284.3, 102.3)
- added C153: 100nF, Capacitor_SMD:C_0603_1608Metric, B.Cu at (37.6, 102.8)
- added C154: 100nF, Capacitor_SMD:C_0603_1608Metric, B.Cu at (73.4, 121.8)
- added C155: 100nF, Capacitor_SMD:C_0603_1608Metric, B.Cu at (91.4, 122.3)
- added C156: 100nF, Capacitor_SMD:C_0603_1608Metric, B.Cu at (110.5, 122.3)
- added C157: 100nF, Capacitor_SMD:C_0603_1608Metric, B.Cu at (129.5, 122.3)
- added C158: 100nF, Capacitor_SMD:C_0603_1608Metric, B.Cu at (148.6, 122.3)
- added C159: 100nF, Capacitor_SMD:C_0603_1608Metric, B.Cu at (167.6, 122.3)
- added C160: 100nF, Capacitor_SMD:C_0603_1608Metric, B.Cu at (186.7, 122.3)
- added C161: 100nF, Capacitor_SMD:C_0603_1608Metric, B.Cu at (205.7, 122.3)
- added C162: 100nF, Capacitor_SMD:C_0603_1608Metric, B.Cu at (224.8, 122.3)
- added C163: 100nF, Capacitor_SMD:C_0603_1608Metric, B.Cu at (243.8, 122.3)
- added C164: 100nF, Capacitor_SMD:C_0603_1608Metric, B.Cu at (279.5, 122.3)
- added C165: 100nF, Capacitor_SMD:C_0603_1608Metric, B.Cu at (341.0, 122.3)
- added C166: 100nF, Capacitor_SMD:C_0603_1608Metric, B.Cu at (31.9, 141.4)
- added C167: 100nF, Capacitor_SMD:C_0603_1608Metric, B.Cu at (55.7, 141.4)
- added C168: 100nF, Capacitor_SMD:C_0603_1608Metric, B.Cu at (79.5, 140.4)
- added C169: 100nF, Capacitor_SMD:C_0603_1608Metric, B.Cu at (41.4, 122.3)
- added C170: 100nF, Capacitor_SMD:C_0603_1608Metric, B.Cu at (150.9, 141.4)
- added C171: 100nF, Capacitor_SMD:C_0603_1608Metric, B.Cu at (223.4, 140.9)
- added C172: 100nF, Capacitor_SMD:C_0603_1608Metric, B.Cu at (246.2, 137.9)
- added C173: 100nF, Capacitor_SMD:C_0603_1608Metric, B.Cu at (271.0, 140.9)
- added C174: 100nF, Capacitor_SMD:C_0603_1608Metric, B.Cu at (292.3, 136.4)
- added C175: 100nF, Capacitor_SMD:C_0603_1608Metric, B.Cu at (321.9, 141.4)
- added C176: 100nF, Capacitor_SMD:C_0603_1608Metric, B.Cu at (340.9, 141.4)
- added C177: 100nF, Capacitor_SMD:C_0603_1608Metric, B.Cu at (360.0, 140.4)
- added C178: 100nF, Capacitor_SMD:C_0603_1608Metric, B.Cu at (274.1, 48.6)
- added C179: 100nF, Capacitor_SMD:C_0603_1608Metric, B.Cu at (288.2, 42.1)
- added C3: 100nF, Capacitor_SMD:C_0603_1608Metric, F.Cu at (331.5, 58.0)
- added C4: 100nF, Capacitor_SMD:C_0603_1608Metric, F.Cu at (336.5, 64.0)
- added C5: 100nF, Capacitor_SMD:C_0603_1608Metric, F.Cu at (365.2, 50.8)
- added C6: 1uF, Capacitor_SMD:C_0805_2012Metric, F.Cu at (351.5, 76.0)
- added C7: 22uF, Capacitor_SMD:C_1206_3216Metric, F.Cu at (357.0, 82.5)
- added C9: 10nF, Capacitor_SMD:C_0603_1608Metric, F.Cu at (356.0, 64.8)
- added Q2: BSS138LT1G, Package_TO_SOT_SMD:SOT-23, F.Cu at (358.5, 46.0)
- added R10: 2.2k, Resistor_SMD:R_0603_1608Metric, F.Cu at (354.0, 42.0)
- added R11: 10k, Resistor_SMD:R_0603_1608Metric, F.Cu at (365.0, 48.0)
- added R12: 160k, Resistor_SMD:R_0603_1608Metric, F.Cu at (361.0, 77.0)
- added R2: 330, Resistor_SMD:R_0603_1608Metric, F.Cu at (331.5, 66.0)
- added R3: 100k, Resistor_SMD:R_0603_1608Metric, F.Cu at (327.0, 59.0)
- added R4: 100k, Resistor_SMD:R_0603_1608Metric, F.Cu at (328.0, 64.0)
- added R5: 2.2k, Resistor_SMD:R_0603_1608Metric, F.Cu at (361.0, 74.0)
- added R6: 2.2k, Resistor_SMD:R_0603_1608Metric, F.Cu at (354.5, 71.0)
- added R7: 4.7k, Resistor_SMD:R_0603_1608Metric, F.Cu at (350.0, 46.0)
- added R8: 4.7k, Resistor_SMD:R_0603_1608Metric, F.Cu at (353.0, 48.0)
- added R9: 10k, Resistor_SMD:R_0603_1608Metric, F.Cu at (361.0, 43.0)
- added U2: SN74LVC1T45DBVR, Package_TO_SOT_SMD:SOT-23-6, F.Cu at (334.5, 61.0)
- added U3: TPS2553DBVR, Package_TO_SOT_SMD:SOT-23-6, F.Cu at (357.0, 77.0)
- added U4: PCA9536DR, Package_SO:SOIC-8_3.9x4.9mm_P1.27mm, F.Cu at (360.5, 55.0)
- added U5: TPS22918DBVR, Package_TO_SOT_SMD:SOT-23-6, F.Cu at (354.0, 68.0)
- A1: value RaspberryPi_Pico -> Raspberry Pi Pico W; footprint Module:RaspberryPi_Pico_Common_THT -> KeyboardVerified:RaspberryPi_Pico_Common_THT_Bare_W
- C1, C2: value 4.7 uF -> 10uF
- SW10, SW11, SW13, SW14, SW15, SW16, SW17, SW18, SW19, SW2, SW20, SW21, SW22, SW23, SW24, SW25, SW26, SW27, SW29, SW3, SW30, SW31, SW32, SW33, SW34, SW35, SW36, SW37, SW38, SW39, SW4, SW40, SW41, SW42, SW43, SW44, SW45, SW46, SW47, SW48, SW49, SW5, SW50, SW51, SW52, SW53, SW54, SW55, SW57, SW58, SW6, SW60, SW61, SW62, SW63, SW64, SW65, SW66, SW67, SW68, SW69, SW7, SW71, SW72, SW73, SW74, SW77, SW79, SW8, SW80, SW81, SW82, SW9, SW90, SW91, SW92, SW93, SW94, SW95: footprint KeyBoardLibrary:SW_MX_1u -> KeyboardVerified:SW_MX_1u
- SW12: footprint KeyBoardLibrary:SW_MX_1u -> KeyboardVerified:SW_MX_1u_RGB_Clearance
Connections:
- net Net-(U1-PROG) renamed /CHG_PROG
- C1 pad 1: +5V -> CHG_5V
- RGB1 pad 2: RGB_DATA -> RGB_DIN_5V
- RGB1 pad 3: +5V -> RGB_5V
- RGB10 pad 3: +5V -> RGB_5V
- RGB11 pad 3: +5V -> RGB_5V
- RGB12 pad 3: +5V -> RGB_5V
- RGB13 pad 3: +5V -> RGB_5V
- RGB14 pad 3: +5V -> RGB_5V
- RGB15 pad 3: +5V -> RGB_5V
- RGB16 pad 3: +5V -> RGB_5V
- RGB17 pad 3: +5V -> RGB_5V
- RGB18 pad 3: +5V -> RGB_5V
- RGB19 pad 3: +5V -> RGB_5V
- RGB2 pad 3: +5V -> RGB_5V
- RGB20 pad 3: +5V -> RGB_5V
- RGB21 pad 3: +5V -> RGB_5V
- RGB22 pad 3: +5V -> RGB_5V
- RGB23 pad 3: +5V -> RGB_5V
- RGB24 pad 3: +5V -> RGB_5V
- RGB25 pad 3: +5V -> RGB_5V
- RGB26 pad 3: +5V -> RGB_5V
- RGB27 pad 3: +5V -> RGB_5V
- RGB3 pad 3: +5V -> RGB_5V
- RGB31 pad 3: +5V -> RGB_5V
- RGB32 pad 3: +5V -> RGB_5V
- RGB33 pad 3: +5V -> RGB_5V
- RGB34 pad 3: +5V -> RGB_5V
- RGB35 pad 3: +5V -> RGB_5V
- RGB36 pad 3: +5V -> RGB_5V
- RGB37 pad 3: +5V -> RGB_5V
- RGB38 pad 3: +5V -> RGB_5V
- RGB39 pad 3: +5V -> RGB_5V
- RGB4 pad 3: +5V -> RGB_5V
- RGB40 pad 3: +5V -> RGB_5V
- RGB41 pad 3: +5V -> RGB_5V
- RGB42 pad 3: +5V -> RGB_5V
- RGB43 pad 3: +5V -> RGB_5V
- RGB46 pad 3: +5V -> RGB_5V
- RGB47 pad 3: +5V -> RGB_5V
- RGB48 pad 3: +5V -> RGB_5V
- RGB49 pad 3: +5V -> RGB_5V
- RGB5 pad 3: +5V -> RGB_5V
- RGB50 pad 3: +5V -> RGB_5V
- RGB51 pad 3: +5V -> RGB_5V
- RGB52 pad 3: +5V -> RGB_5V
- RGB53 pad 3: +5V -> RGB_5V
- RGB54 pad 3: +5V -> RGB_5V
- RGB55 pad 3: +5V -> RGB_5V
- RGB56 pad 3: +5V -> RGB_5V
- RGB57 pad 3: +5V -> RGB_5V
- RGB58 pad 3: +5V -> RGB_5V
- RGB59 pad 3: +5V -> RGB_5V
- RGB6 pad 3: +5V -> RGB_5V
- RGB60 pad 3: +5V -> RGB_5V
- RGB61 pad 3: +5V -> RGB_5V
- RGB62 pad 3: +5V -> RGB_5V
- RGB63 pad 3: +5V -> RGB_5V
- RGB64 pad 3: +5V -> RGB_5V
- RGB65 pad 3: +5V -> RGB_5V
- RGB66 pad 3: +5V -> RGB_5V
- RGB67 pad 3: +5V -> RGB_5V
- RGB68 pad 3: +5V -> RGB_5V
- RGB69 pad 3: +5V -> RGB_5V
- RGB7 pad 3: +5V -> RGB_5V
- RGB70 pad 3: +5V -> RGB_5V
- RGB71 pad 3: +5V -> RGB_5V
- RGB72 pad 3: +5V -> RGB_5V
- RGB73 pad 3: +5V -> RGB_5V
- RGB74 pad 3: +5V -> RGB_5V
- RGB75 pad 3: +5V -> RGB_5V
- RGB76 pad 3: +5V -> RGB_5V
- RGB77 pad 3: +5V -> RGB_5V
- RGB78 pad 3: +5V -> RGB_5V
- RGB79 pad 3: +5V -> RGB_5V
- RGB8 pad 3: +5V -> RGB_5V
- RGB80 pad 3: +5V -> RGB_5V
- RGB81 pad 3: +5V -> RGB_5V
- RGB82 pad 3: +5V -> RGB_5V
- RGB83 pad 3: +5V -> RGB_5V
- RGB84 pad 3: +5V -> RGB_5V
- RGB9 pad 3: +5V -> RGB_5V
- U1 pad 1: unconnected-(U1-STAT-Pad1) -> (no net)
- U1 pad 4: +5V -> CHG_5V
Routing:
- net RGB_5V: track 0.00 -> 789.6 mm, vias 0 -> 93
- net +5V: track 693.0 -> 90.9 mm, vias 73 -> 6
- net RGB_DIN_5V: track 0.00 -> 396.6 mm, vias 0 -> 7
- net RGB_DATA: track 355.3 -> 37.3 mm
- net GND: track 2928.5 -> 3109.2 mm, vias 28 -> 118
- net /COL3: track 953.7 -> 875.4 mm, vias 12 -> 11
- net +3V3: track 27.2 -> 102.0 mm, vias 1 -> 10
- net RGB_ENABLE: track 0.00 -> 49.0 mm
- net RGB_FAULT_N: track 0.00 -> 36.2 mm
- net /OLED_SCL: track 25.9 -> 60.5 mm, vias 2 -> 4
- net /COL12: track 233.6 -> 267.8 mm, vias 1 -> 7
- net /OLED_SDA: track 18.0 -> 51.1 mm, vias 0 -> 3
- net CHG_ENABLE: track 0.00 -> 24.9 mm, vias 0 -> 2
- net CHG_5V: track 0.00 -> 21.1 mm, vias 0 -> 2
- net USB_PRESENT_N: track 0.00 -> 16.3 mm, vias 0 -> 4
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- added copper zone on F.Cu, net GND
- added copper zone on B.Cu, net RGB_5V
- removed copper zone on B.Cu, net +5V
Other:
- outline, holes or cut-outs redrawn
