File: pcb/keeb_pcb.kicad_sch (KiCad schematic)
At the start: 242 parts, among them J1 Conn_01x04, SW10 SW_Push, SW11 SW_Push, SW12 SW_Push, SW13 SW_Push, SW14 SW_Push, SW15 SW_Push, SW16 SW_Push, SW17 SW_Push, SW18 SW_Push, SW19 SW_Push, SW2 SW_Push, SW20 SW_Push, SW21 SW_Push, SW22 SW_Push, SW23 SW_Push, SW24 SW_Push, SW25 SW_Push, SW26 SW_Push, SW27 SW_Push, SW29 SW_Push, SW3 SW_Push, SW30 SW_Push, SW31 SW_Push, SW32 SW_Push, SW33 SW_Push, SW34 SW_Push, SW35 SW_Push, SW36 SW_Push, SW37 SW_Push, SW38 SW_Push, SW39 SW_Push, SW4 SW_Push, SW40 SW_Push, SW41 SW_Push, SW42 SW_Push, SW43 SW_Push, SW44 SW_Push, SW45 SW_Push, SW46 SW_Push, SW47 SW_Push, SW48 SW_Push, SW49 SW_Push, SW5 SW_Push, SW50 SW_Push, SW51 SW_Push, SW52 SW_Push, SW53 SW_Push, SW54 SW_Push, SW55 SW_Push, SW57 SW_Push, SW58 SW_Push, SW6 SW_Push, SW60 SW_Push, SW61 SW_Push, SW62 SW_Push, SW63 SW_Push, SW64 SW_Push, SW65 SW_Push, SW66 SW_Push, SW67 SW_Push, SW68 SW_Push, SW69 SW_Push, SW7 SW_Push, SW71 SW_Push, SW72 SW_Push, SW73 SW_Push, SW74 SW_Push, SW77 SW_Push, SW79 SW_Push, SW8 SW_Push, SW80 SW_Push, SW81 SW_Push, SW82 SW_Push, SW9 SW_Push, SW90 SW_Push, SW91 SW_Push, SW92 SW_Push, SW93 SW_Push

Commit message: Added new PCB files and removed old journal entries.
Connections:
- net RGB_D27: now also RGB31.2 (DIN)
- net RGB_D31: now also RGB31.4 (DOUT)
- net RGB_D43: now also RGB46.2 (DIN)
- net RGB_D46: now also RGB47.2 (DIN)
- net RGB_D47: now also RGB47.4 (DOUT)
- net RGB_D48: now also RGB49.2 (DIN)
- net RGB_D82: no longer names the net of RGB82.4 (DOUT)
- no-connect marks 6 -> 7

Commit message: Updated with Log 6
Parts:
- added C1, C2: 4.7 uF, Capacitor_SMD:C_0805_2012Metric, symbol Device:C
- added D1: SS14, Diode_SMD:D_SMA, symbol Device:D_Schottky
- added D94, D95: 1N4148, Diode_THT:D_DO-35_SOD27_P7.62mm_Horizontal, symbol Diode:1N4148
- added JST_1: J_BAT, Connector_JST:JST_PH_B2B-PH-K_1x02_P2.00mm_Vertical, symbol Connector_Generic:Conn_01x02
- added R1: 10k, Resistor_SMD:R_0805_2012Metric, symbol Device:R
- added RGB83, RGB84: SK6812MINI-E, LED_SMD:LED_SK6812MINI-E_3.2x2.8mm_P1.5mm_ReverseMount, symbol LED:SK6812MINI-E
- added SW1: SW_PWR, Button_Switch_THT:SW_Slide-03_Wuerth-WS-SLTV_10x2.5x6.4_P2.54mm, symbol Switch:SW_SPST
- added SW94: Programmable 1, KeyBoardLibrary:SW_MX_1u, symbol Switch:SW_Push
- added SW95: Programmable 2, KeyBoardLibrary:SW_MX_1u, symbol Switch:SW_Push
- added U1: MCP73831-2-OT, Package_TO_SOT_SMD:SOT-23-5, symbol Battery_Management:MCP73831-2-OT
- J1: footprint (none) -> Connector_PinHeader_2.54mm:PinHeader_1x04_P2.54mm_Vertical
Connections:
- net +5V: now also C1.1, RGB83.3 (VDD), RGB84.3 (VDD), U1.4 (V_{DD}); no longer J1.2 (Pin_2)
- net COL5: now also SW94.1
- net COL6: now also SW95.1
- net GND: now also C1.2, C2.1, JST_1.2 (Pin_2), R1.1, RGB83.1 (VSS), RGB84.1 (VSS), U1.2 (V_{SS})
- net RGB_D13: now also RGB84.4 (DOUT); no longer RGB13.4 (DOUT)
- net ROW5: now also D94.1 (K), D95.1 (K)
- net +3V3: now reaches A1.36 (3V3)
- net +3V3: now also J1.2 (Pin_2)
- net at A1.39 (VSYS): now also D1.1 (K)
- new net: R1.2, U1.5 (PROG)
- new net: D95.2 (A), SW95.2
- new net: D94.2 (A), SW94.2
- new net BAT+: C2.2, JST_1.1 (Pin_1), SW1.2 (B), U1.3 (V_{BAT})
- new net BAT_SW: D1.2 (A), SW1.1 (A)
- new net RGB_NEW_A: RGB13.4 (DOUT), RGB83.2 (DIN)
- new net RGB_NEW_B: RGB83.4 (DOUT), RGB84.2 (DIN)
- no-connect marks 7 -> 6
Other:
- moved on the sheet: D28, ENC1

Commit message: Publish checked keyboard hardware, fabrication files and repaired case source
Parts:
- added C10, C6: 1uF, Capacitor_SMD:C_0805_2012Metric, symbol KeyboardPower:C
- added C101, C102, C103, C104, C105, C106, C107, C108, C109, C110, C111, C112, C113, C114, C115, C116, C117, C118, C119, C120, C121, C122, C123, C124, C125, C126, C127, C128, C129, C130, C131, C132, C133, C134, C135, C136, C137, C138, C139, C140, C141, C142, C143, C144, C145, C146, C147, C148, C149, C150, C151, C152, C153, C154, C155, C156, C157, C158, C159, C160, C161, C162, C163, C164, C165, C166, C167, C168, C169, C170, C171, C172, C173, C174, C175, C176, C177, C178, C179, C3, C4, C5: 100nF, Capacitor_SMD:C_0603_1608Metric, symbol KeyboardPower:C
- added C7: 22uF, Capacitor_SMD:C_1206_3216Metric, symbol KeyboardPower:C
- added C9: 10nF, Capacitor_SMD:C_0603_1608Metric, symbol KeyboardPower:C
- added Q2: BSS138LT1G, Package_TO_SOT_SMD:SOT-23, symbol KeyboardPower:BSS138
- added R10, R5, R6: 2.2k, Resistor_SMD:R_0603_1608Metric, symbol KeyboardPower:R
- added R11, R9: 10k, Resistor_SMD:R_0603_1608Metric, symbol KeyboardPower:R
- added R12: 160k, Resistor_SMD:R_0603_1608Metric, symbol KeyboardPower:R
- added R2: 330, Resistor_SMD:R_0603_1608Metric, symbol KeyboardPower:R
- added R3, R4: 100k, Resistor_SMD:R_0603_1608Metric, symbol KeyboardPower:R
- added R7, R8: 4.7k, Resistor_SMD:R_0603_1608Metric, symbol KeyboardPower:R
- added U2: SN74LVC1T45DBVR, Package_TO_SOT_SMD:SOT-23-6, symbol KeyboardPower:SN74LVC1T45
- added U3: TPS2553DBVR, Package_TO_SOT_SMD:SOT-23-6, symbol KeyboardPower:TPS2553
- added U4: PCA9536DR, Package_SO:SOIC-8_3.9x4.9mm_P1.27mm, symbol KeyboardPower:PCA9536
- added U5: TPS22918DBVR, Package_TO_SOT_SMD:SOT-23-6, symbol KeyboardPower:TPS22918
- A1: value RaspberryPi_Pico -> Raspberry Pi Pico W; footprint Module:RaspberryPi_Pico_Common_THT -> KeyboardVerified:RaspberryPi_Pico_Common_THT_Bare_W
- C1, C2: value 4.7 uF -> 10uF
- SW10, SW11, SW13, SW14, SW15, SW16, SW17, SW18, SW19, SW2, SW20, SW21, SW22, SW23, SW24, SW25, SW26, SW27, SW29, SW3, SW30, SW31, SW32, SW33, SW34, SW35, SW36, SW37, SW38, SW39, SW4, SW40, SW41, SW42, SW43, SW44, SW45, SW46, SW47, SW48, SW49, SW5, SW50, SW51, SW52, SW53, SW54, SW55, SW57, SW58, SW6, SW60, SW61, SW62, SW63, SW64, SW65, SW66, SW67, SW68, SW69, SW7, SW71, SW72, SW73, SW74, SW77, SW79, SW8, SW80, SW81, SW82, SW9, SW90, SW91, SW92, SW93: footprint PCM_marbastlib-mx:SW_MX_1u -> KeyboardVerified:SW_MX_1u
- SW12: footprint PCM_marbastlib-mx:SW_MX_1u -> KeyboardVerified:SW_MX_1u_RGB_Clearance
- SW94, SW95: footprint KeyBoardLibrary:SW_MX_1u -> KeyboardVerified:SW_MX_1u
Connections:
- net +3V3: now also C3.1, C5.1, R11.1, R7.1, R8.1, R9.1, U2.1 (VCCA), U2.5 (DIR), U4.8 (VCC)
- net +5V: now also C10.1, C6.1, Q2.1 (G), R10.1, U3.1 (IN), U5.1 (VIN); no longer C1.1, RGB1.3 (VDD), RGB10.3 (VDD), RGB11.3 (VDD), RGB12.3 (VDD), RGB13.3 (VDD), RGB14.3 (VDD), RGB15.3 (VDD), RGB16.3 (VDD), RGB17.3 (VDD), RGB18.3 (VDD), RGB19.3 (VDD), RGB2.3 (VDD), RGB20.3 (VDD), RGB21.3 (VDD), RGB22.3 (VDD), RGB23.3 (VDD), RGB24.3 (VDD), RGB25.3 (VDD), RGB26.3 (VDD), RGB27.3 (VDD), RGB3.3 (VDD), RGB31.3 (VDD), RGB32.3 (VDD), RGB33.3 (VDD), RGB34.3 (VDD), RGB35.3 (VDD), RGB36.3 (VDD), RGB37.3 (VDD), RGB38.3 (VDD), RGB39.3 (VDD), RGB4.3 (VDD), RGB40.3 (VDD), RGB41.3 (VDD), RGB42.3 (VDD), RGB43.3 (VDD), RGB46.3 (VDD), RGB47.3 (VDD), RGB48.3 (VDD), RGB49.3 (VDD), RGB5.3 (VDD), RGB50.3 (VDD), RGB51.3 (VDD), RGB52.3 (VDD), RGB53.3 (VDD), RGB54.3 (VDD), RGB55.3 (VDD), RGB56.3 (VDD), RGB57.3 (VDD), RGB58.3 (VDD), RGB59.3 (VDD), RGB6.3 (VDD), RGB60.3 (VDD), RGB61.3 (VDD), RGB62.3 (VDD), RGB63.3 (VDD), RGB64.3 (VDD), RGB65.3 (VDD), RGB66.3 (VDD), RGB67.3 (VDD), RGB68.3 (VDD), RGB69.3 (VDD), RGB7.3 (VDD), RGB70.3 (VDD), RGB71.3 (VDD), RGB72.3 (VDD), RGB73.3 (VDD), RGB74.3 (VDD), RGB75.3 (VDD), RGB76.3 (VDD), RGB77.3 (VDD), RGB78.3 (VDD), RGB79.3 (VDD), RGB8.3 (VDD), RGB80.3 (VDD), RGB81.3 (VDD), RGB82.3 (VDD), RGB83.3 (VDD), RGB84.3 (VDD), RGB9.3 (VDD), U1.4 (V_{DD})
- net GND: now also C10.2, C101.2, C102.2, C103.2, C104.2, C105.2, C106.2, C107.2, C108.2, C109.2, C110.2, C111.2, C112.2, C113.2, C114.2, C115.2, C116.2, C117.2, C118.2, C119.2, C120.2, C121.2, C122.2, C123.2, C124.2, C125.2, C126.2, C127.2, C128.2, C129.2, C130.2, C131.2, C132.2, C133.2, C134.2, C135.2, C136.2, C137.2, C138.2, C139.2, C140.2, C141.2, C142.2, C143.2, C144.2, C145.2, C146.2, C147.2, C148.2, C149.2, C150.2, C151.2, C152.2, C153.2, C154.2, C155.2, C156.2, C157.2, C158.2, C159.2, C160.2, C161.2, C162.2, C163.2, C164.2, C165.2, C166.2, C167.2, C168.2, C169.2, C170.2, C171.2, C172.2, C173.2, C174.2, C175.2, C176.2, C177.2, C178.2, C179.2, C3.2, C4.2, C5.2, C6.2, C7.2, C9.2, Q2.2 (S), R10.2, R12.2, R3.2, R4.2, R5.2, R6.2, U2.2 (GND), U3.2 (GND), U4.4 (GND), U5.2 (GND)
- net OLED_SCL: now also R7.2, U4.6 (SCL)
- net OLED_SDA: now also R8.2, U4.7 (SDA)
- net RGB_DATA: now also R3.1, U2.3 (A); no longer RGB1.2 (DIN)
- net CHG_PROG: now reaches R1.2, U1.5 (PROG)
- new net CHG_5V: C1.1, U1.4 (V_{DD}), U5.5 (QOD), U5.6 (VOUT)
- new net CHG_ENABLE: R6.1, U4.2 (IO1), U5.3 (ON)
- new net CHG_SLEW: C9.1, U5.4 (CT)
- new net RGB_5V: C101.1, C102.1, C103.1, C104.1, C105.1, C106.1, C107.1, C108.1, C109.1, C110.1, C111.1, C112.1, C113.1, C114.1, C115.1, C116.1, C117.1, C118.1, C119.1, C120.1, C121.1, C122.1, C123.1, C124.1, C125.1, C126.1, C127.1, C128.1, C129.1, C130.1, C131.1, C132.1, C133.1, C134.1, C135.1, C136.1, C137.1, C138.1, C139.1, C140.1, C141.1, C142.1, C143.1, C144.1, C145.1, C146.1, C147.1, C148.1, C149.1, C150.1, C151.1, C152.1, C153.1, C154.1, C155.1, C156.1, C157.1, C158.1, C159.1, C160.1, C161.1, C162.1, C163.1, C164.1, C165.1, C166.1, C167.1, C168.1, C169.1, C170.1, C171.1, C172.1, C173.1, C174.1, C175.1, C176.1, C177.1, C178.1, C179.1, C4.1, C7.1, RGB1.3 (VDD), RGB10.3 (VDD), RGB11.3 (VDD), RGB12.3 (VDD), RGB13.3 (VDD), RGB14.3 (VDD), RGB15.3 (VDD), RGB16.3 (VDD), RGB17.3 (VDD), RGB18.3 (VDD), RGB19.3 (VDD), RGB2.3 (VDD), RGB20.3 (VDD), RGB21.3 (VDD), RGB22.3 (VDD), RGB23.3 (VDD), RGB24.3 (VDD), RGB25.3 (VDD), RGB26.3 (VDD), RGB27.3 (VDD), RGB3.3 (VDD), RGB31.3 (VDD), RGB32.3 (VDD), RGB33.3 (VDD), RGB34.3 (VDD), RGB35.3 (VDD), RGB36.3 (VDD), RGB37.3 (VDD), RGB38.3 (VDD), RGB39.3 (VDD), RGB4.3 (VDD), RGB40.3 (VDD), RGB41.3 (VDD), RGB42.3 (VDD), RGB43.3 (VDD), RGB46.3 (VDD), RGB47.3 (VDD), RGB48.3 (VDD), RGB49.3 (VDD), RGB5.3 (VDD), RGB50.3 (VDD), RGB51.3 (VDD), RGB52.3 (VDD), RGB53.3 (VDD), RGB54.3 (VDD), RGB55.3 (VDD), RGB56.3 (VDD), RGB57.3 (VDD), RGB58.3 (VDD), RGB59.3 (VDD), RGB6.3 (VDD), RGB60.3 (VDD), RGB61.3 (VDD), RGB62.3 (VDD), RGB63.3 (VDD), RGB64.3 (VDD), RGB65.3 (VDD), RGB66.3 (VDD), RGB67.3 (VDD), RGB68.3 (VDD), RGB69.3 (VDD), RGB7.3 (VDD), RGB70.3 (VDD), RGB71.3 (VDD), RGB72.3 (VDD), RGB73.3 (VDD), RGB74.3 (VDD), RGB75.3 (VDD), RGB76.3 (VDD), RGB77.3 (VDD), RGB78.3 (VDD), RGB79.3 (VDD), RGB8.3 (VDD), RGB80.3 (VDD), RGB81.3 (VDD), RGB82.3 (VDD), RGB83.3 (VDD), RGB84.3 (VDD), RGB9.3 (VDD), U2.6 (VCCB), U3.6 (OUT)
- new net RGB_BUFFER_OUT: R2.1, U2.4 (B)
- new net RGB_DIN_5V: R2.2, R4.1, RGB1.2 (DIN)
- new net RGB_ENABLE: R5.1, U3.3 (EN), U4.1 (IO0)
- new net RGB_FAULT_N: R11.2, U3.4 (FAULT_N), U4.5 (IO3)
- new net RGB_ILIM: R12.1, U3.5 (ILIM)
- new net USB_PRESENT_N: Q2.3 (D), R9.2, U4.3 (IO2)
